File: wait_request.kicad_pcb (KiCad board)
At the start: 2 copper layers, 85 x 65 mm, 27 parts, among them J1 WAIT Delay Selecter, X1 Power, X2 Address, X3 Data, X4 Mode, X5 Control, X6 Clock

Commit message: Update
Parts:
- removed the R2 at (86.0, 112.1)
- DD1: value 555ЛА1 (74LS20) -> 555ЛА2 (74LS30)
- moved REF** 150.9 mm to (92.2, 121.9)
- moved REF** 120.2 mm to (92.2, 84.6)
- moved REF** 84.4 mm to (129.7, 100.0), turned to 180 degrees
- renumbered DD3 to DD2, DD2 to DD3, R3 to R2, R4 to R3, R5 to R4
Connections:
- DD1 pad 10: /~{IOR} -> (no net)
- DD1 pad 11: (no net) -> /~{MEMR}
- DD1 pad 12: Net-(DD1-Pad12) -> /~{IOR}
- DD1 pad 13: Net-(DD1-Pad12) -> (no net)
- DD1 pad 3: (no net) -> /~{MEMW}
- DD1 pad 4: /~{MEMW} -> Net-(DD1-Pad4)
- DD1 pad 5: Net-(DD1-Pad5) -> Net-(DD1-Pad4)
- DD1 pad 6: Net-(DD1-Pad6) -> Net-(DD1-Pad4)
- DD1 pad 8: Net-(DD1-Pad8) -> Net-(DD2-~{R})
- DD1 pad 9: /~{MEMR} -> (no net)
- DD2 pad 8: /F2TTL -> Net-(DD2-CK)
- DD2 pad 9: Net-(DD3-~{R}) -> Net-(DD2-~{R})
- DD3 pad 1: Net-(DD1-Pad6) -> GND
- DD3 pad 11: unconnected-(DD2-Pad11) -> Net-(DD2-CK)
- DD3 pad 12: GND -> /F2TTL
- DD3 pad 2: Net-(DD1-Pad8) -> GND
- DD3 pad 3: Net-(DD3-~{R}) -> unconnected-(DD3-Pad3)
- R1 pad 1: Net-(DD1-Pad5) -> Net-(DD1-Pad4)
Routing:
- net Net-(DD2-~{R}): track 0.00 -> 71.7 mm
- net Net-(DD3-~{R}): track 51.2 -> 0.00 mm
- net Net-(DD2-CK): track 0.00 -> 43.2 mm, vias 0 -> 1
- net Net-(DD1-Pad8): track 24.6 -> 0.00 mm
- net Net-(DD1-Pad6): track 17.0 -> 0.00 mm
- net /F2TTL: track 61.4 -> 46.9 mm, vias 0 -> 2
- net Net-(DD1-Pad4): track 0.00 -> 7.58 mm
- net Net-(DD1-Pad12): track 5.06 -> 0.00 mm
- net Net-(DD1-Pad5): track 2.40 -> 0.00 mm
- net /~{MEMR}: track 16.5 -> 18.6 mm
- net /~{IOR}: track 16.5 -> 18.6 mm
- net /~{MEMW}: track 24.1 -> 26.2 mm
- net /~{IOW}: track 25.2 -> 26.2 mm
- net /~{WRQ}: track 60.1 -> 59.2 mm
- net /~{INTA}: track 24.1 -> 24.7 mm
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Other:
- board text added: "555ЛА2"
- board text added: "v.1.1 07/08/2026"
- board text removed: "555ЛА1"
- board text removed: "555ЛИ1"
- board text removed: "v.1.0 25/03/2026"
