File: wait_request.kicad_sch (KiCad schematic)
At the start: 24 parts, among them J1 WAIT Delay Selecter, X1 Power, X2 Address, X3 Data, X4 Mode, X5 Control, X6 Clock

Commit message: Update
Parts:
- removed DD1: 555ЛА1 (74LS20), Package_DIP:DIP-14_W7.62mm_Socket_LongPads, symbol 74xx:74LS20
- removed R2: 1k, Resistor_SMD:R_0805_2012Metric_Pad1.20x1.40mm_HandSolder, symbol Device:R
- added DD1: 555ЛА2 (74LS30), Package_DIP:DIP-14_W7.62mm_Socket_LongPads, symbol 74xx:74LS30
- renumbered C5 to C3, C3 to C4, C4 to C5, C8 to C6, C6 to C7, C7 to C8, DD3 to DD2, DD2 to DD3, R3 to R2, R4 to R3, R5 to R4
Connections:
- net +5: now also DD1.14 (VCC)
- net F2TTL: now also DD3.12; no longer DD2.8 (CK)
- net GND: now also DD3.1, DD3.2, DD1.7 (GND); no longer DD3.12
- net ~{INTA}: now also DD1.1
- net ~{IOR}: now also DD1.12
- net ~{IOW}: now also DD1.2
- net ~{MEMR}: now also DD1.11
- net ~{MEMW}: now also DD1.3
- net at DD3.3: no longer DD2.9 (~{R})
- net at R1.1: now also DD1.4, DD1.5, DD1.6
- net at DD3.11: now also DD2.8 (CK)
- new net: DD1.8, DD2.9 (~{R})
Other:
- moved on the sheet: DD3A, DD3C, DD3D
